File: _autosave-CRVFCU.kicad_sch (KiCad schematic)
At the start: 150 parts, among them J1 TagConnect_TC2030, J3 USB_C_Receptacle_USB2.0_16P, J4 Micro_SD_Card_Det2, Q3 DMG2301L, Q4 BC818, Q5 DMG2301L, Q6 DMG2301L, SW1 SW_Omron_B3FS, SW2 SW_Nidec_CAS-120A1, U1 MS5611-01BA, U10 W25Q128JVS, U11 CM1624, U13 USBLC6-2SC6, U14 USBLC6-2SC6, U15 MAX17049, U16 SI7232DN-T1, U17 SN74LV1T34DCK, U2 STM32H747IITx, U3 LIS2MDL, U4 ICM-45686, U5 FXMA108, U6 AP1117-50, U7 AP1117-33, U8 SI7232DN-T1, U9 USBLC6-4SC6, Y1 32.768khz, Y3 32.768khz, Y4 25MHZ

Commit message: completed grouping in pcb, prep for route
Connections:
- net PYO0: now also PYRO_TERM1.4 (Pin_4); no longer PYRO_TERM1.10 (Pin_10)
- net PYO1: now also PYRO_TERM1.5 (Pin_5); no longer PYRO_TERM1.4 (Pin_4)
- net PYO2: now also PYRO_TERM1.8 (Pin_8); no longer PYRO_TERM1.6 (Pin_6)
- net PYO3: now also PYRO_TERM1.9 (Pin_9); no longer PYRO_TERM1.8 (Pin_8)
- net VPYRO: now also PYRO_TERM1.10 (Pin_10), PYRO_TERM1.6 (Pin_6); no longer PYRO_TERM1.5 (Pin_5), PYRO_TERM1.9 (Pin_9)
Changed lines of the file:
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@@
 		)
 	)
-	(label "PYO2"
+	(label "VPYRO"
 		(at 405.13 379.73 0)
 		(effects
@@
 		)
 	)
-	(label "VPYRO"
+	(label "PYO1"
 		(at 406.4 377.19 0)
 		(effects
@@
 		)
 	)
-	(label "VPYRO"
+	(label "PYO3"
 		(at 406.4 387.35 0)
 		(effects
@@
 		)
 	)
-	(label "PYO3"
+	(label "PYO2"
 		(at 405.13 384.81 0)
 		(effects
@@
 		)
 	)
-	(label "PYO0"
+	(label "VPYRO"
 		(at 405.13 389.89 0)
 		(effects
@@
 		)
 	)
-	(label "PYO1"
+	(label "PYO0"
 		(at 405.13 374.65 0)
 		(effects
